Commit message: add realsense mount

File: franka_panda_description/urdf/hand.xacro (robot description, xacro)
@@ -13,5 +13,5 @@
       <visual>
         <geometry>
-          <mesh filename="package://franka_description/meshes/visual/hand.dae"/>
+          <mesh filename="package://moveit_resources_franka_description/meshes/visual/hand.dae"/>
         </geometry>
       </visual>
@@ -63,5 +63,5 @@
       <visual>
         <geometry>
-          <mesh filename="package://franka_description/meshes/visual/finger.dae"/>
+		<mesh filename="package://moveit_resources_franka_panda_description/meshes/visual/finger.dae"/>
         </geometry>
       </visual>
@@ -71,5 +71,5 @@
         <origin xyz="0 0 0" rpy="0 0 ${pi}"/>
         <geometry>
-          <mesh filename="package://franka_description/meshes/visual/finger.dae"/>
+          <mesh filename="package://moveit_resources_franka_panda_description/meshes/visual/finger.dae"/>
         </geometry>
       </visual>

File: franka_panda_description/urdf/panda_arm.urdf.xacro (robot description, xacro)
@@ -2,5 +2,6 @@
 <robot xmlns:xacro="http://www.ros.org/wiki/xacro" name="panda">
   <xacro:arg name="arm_id" default="panda"/> <!-- Name of this panda -->
-  <xacro:arg name="hand" default="false"/> <!-- Should a franka_gripper be mounted at the flange?" -->
+  <xacro:arg name="hand_only" default="false"/> <!-- Should a franka_gripper be mounted at the flange?" -->
+  <xacro:arg name="hand_realsense" default="false"/> <!-- Should a franka_gripper and realsense be mounted at the flange?" -->
   <xacro:arg name="robot_ip" default=""/> <!-- IP address or hostname of the robot" -->
   <xacro:arg name="use_fake_hardware" default="false"/>
@@ -8,7 +9,15 @@
   <xacro:include filename="$(find moveit_resources_franka_panda_description)/urdf/panda_arm.xacro"/>
   <xacro:panda_arm arm_id="$(arg arm_id)" safety_distance="0.03"/>
-  <xacro:if value="$(arg hand)">
+  <xacro:if value="$(arg hand_only)">
     <xacro:include filename="$(find moveit_resources_franka_panda_description)/urdf/hand.xacro"/>
     <xacro:hand ns="$(arg arm_id)" rpy="0 0 ${-pi/4}" connected_to="$(arg arm_id)_link8" safety_distance="0.03"/>
+  </xacro:if>
+  <xacro:if value="$(arg hand_realsense)">
+    <xacro:include filename="$(find moveit_resources_franka_panda_description)/urdf/realsense_mount.xacro"/>
+    <xacro:include filename="$(find realsense2_description)/urdf/_d435.urdf.xacro"/>
+    <xacro:include filename="$(find moveit_resources_franka_panda_description)/urdf/hand.xacro"/>
+    <xacro:realsense_mount parent="panda_link8" xyz="0 0 -0.0025" rpy="${radians(180)} 0 ${radians(180)}"/>
+    <xacro:sensor_d435 parent="camera_link" xyz="0 0 0" rpy="0 ${radians(-90)} ${radians(180)}"/>
+    <xacro:hand ns="$(arg arm_id)" rpy="0 0 ${-pi/4}" connected_to="gripper_link" safety_distance="0.03"/>
   </xacro:if>
   <xacro:include filename="$(find moveit_resources_franka_panda_description)/urdf/panda_arm.ros2_control.xacro"/>

File: franka_panda_description/urdf/panda_arm.xacro (robot description, xacro)
@@ -3,5 +3,5 @@
   <!-- safety_distance: Minimum safety distance in [m] by which the collision volumes are expanded and which is enforced during robot motions -->
   <!-- arm_id: Namespace of the panda arm. Serves to differentiate between arms in case of multiple instances. -->
-  <xacro:macro name="panda_arm" params="arm_id:='panda' description_pkg:='franka_description' connected_to:='' xyz:='0 0 0' rpy:='0 0 0' safety_distance:=0">
+  <xacro:macro name="panda_arm" params="arm_id:='panda' description_pkg:='moveit_resources_franka_panda_description' connected_to:='' xyz:='0 0 0' rpy:='0 0 0' safety_distance:=0">
     <xacro:unless value="${not connected_to}">
       <joint name="${arm_id}_joint_${connected_to}" type="fixed">

Commit message: prevent camera_link unique error

File: franka_panda_description/urdf/hand.xacro (robot description, xacro)
@@ -13,5 +13,5 @@
       <visual>
         <geometry>
-          <mesh filename="package://moveit_resources_franka_description/meshes/visual/hand.dae"/>
+          <mesh filename="package://moveit_resources_franka_panda_description/meshes/visual/hand.dae"/>
         </geometry>
       </visual>

File: franka_panda_description/urdf/panda_arm.urdf.xacro (robot description, xacro)
@@ -17,8 +17,8 @@
     <xacro:include filename="$(find realsense2_description)/urdf/_d435.urdf.xacro"/>
     <xacro:include filename="$(find moveit_resources_franka_panda_description)/urdf/hand.xacro"/>
-    <xacro:realsense_mount parent="panda_link8">
+    <xacro:realsense_mount parent="$(arg arm_id)_link8">
       <origin xyz="0 0 -0.0025" rpy="${radians(180)} 0 ${radians(180)}"/>
     </xacro:realsense_mount>
-    <xacro:sensor_d435 parent="camera_link">
+    <xacro:sensor_d435 parent="camera_link" name="realsense">
       <origin xyz="0 0 0" rpy="0 ${radians(-90)} ${radians(180)}"/>
     </xacro:sensor_d435>

File: franka_panda_description/urdf/realsense_mount.xacro (robot description, xacro)
@@ -2,7 +2,7 @@
 <robot name="realsense_mount" xmlns:xacro="http://ros.org/wiki/xacro">
 	<xacro:macro name="realsense_mount" params="parent *origin">
-		<joint name="arm_joint" type="fixed">
+		<joint name="mount_joint" type="fixed">
 			<parent link="${parent}"/>
-			<child link="arm_link"/>
+			<child link="mount_link"/>
 			<origin xyz="0 0 0.0025" rpy="0 0 0"/>
 		</joint>
@@ -11,5 +11,5 @@
 				<origin xyz="0 0 0" rpy="0 0 0"/>
 				<geometry>
-					<mesh filename="$(find moveit_resources_franka_panda_description)/meshes/collision/realsense_mount.stl" scale="1.0 1.0 1.0"/>
+					<mesh filename="package://moveit_resources_franka_panda_description/meshes/collision/realsense_mount.stl" scale="1.0 1.0 1.0"/>
 				</geometry>
 			</visual>
