Commit message: add launch file

File: franka_panda_description/urdf/franka_realsense.urdf (robot description, URDF)
Before this commit: robot panda, 9 links, 8 joints
Links:
- added link camera_link
- added link gripper_link
- added link mount_link; visual mesh filename=/home/peter/Code/ros/panda_stacking_demo/install/moveit_res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 scale=1.0 1.0 1.0
- added link panda_hand; collision cylinder length=0.1 radius=0.05; collision cylinder length=0.1 radius=0.07
- added link panda_hand_tcp
- added link panda_leftfinger; visual mesh filename=package://moveit_resources_franka_panda_description/meshes/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
- added link panda_rightfinger; visual mesh filename=package://moveit_resources_franka_panda_description/meshes/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
- added link realsense_bottom_screw_frame
- added link realsense_link, mass 0.072; collision box size=0.02505 0.09 0.025; visual mesh filename=package://realsense2_description/meshes/d435.dae
Joints:
- added joint arm_joint: type fixed, parent panda_link8, child arm_link, origin xyz=0 0 0.0025 rpy=0 0 0
- added joint camera_joint: type fixed, parent mount_link, child camera_link, origin xyz=0.06 0 0 rpy=0 0 0
- added joint gripper_joint: type fixed, parent mount_link, child gripper_link, origin xyz=0 0 -0.0025 rpy=0 0 0
- added joint panda_finger_joint1: type prismatic, parent panda_hand, child panda_leftfinger, origin xyz=0 0 0.0584 rpy=0 0 0, axis 0 1 0, limit lower=0.0 upper=0.04 effort=20 velocity=0.2
- added joint panda_finger_joint2: type prismatic, parent panda_hand, child panda_rightfinger, origin xyz=0 0 0.0584 rpy=0 0 0, axis 0 -1 0, limit lower=0.0 upper=0.04 effort=20 velocity=0.2, mimic joint=panda_finger_joint1
- added joint panda_hand_joint: type fixed, parent gripper_link, child panda_hand, origin xyz=0 0 0 rpy=0 0 -0.7853981633974483
- added joint panda_hand_tcp_joint: type fixed, parent panda_hand, child panda_hand_tcp, origin xyz=0 0 0.1034 rpy=0 0 0
- added joint realsense_joint: type fixed, parent camera_link, child realsense_bottom_screw_frame, origin xyz=0 0 0 rpy=0 -1.5707963267948966 3.141592653589793
- added joint realsense_link_joint: type fixed, parent realsense_bottom_screw_frame, child realsense_link, origin xyz=0.010600000000000002 0.0175 0.0125 rpy=0 0 0

File: franka_panda_description/urdf/panda_arm.urdf.xacro (robot description, xacro)
@@ -11,5 +11,5 @@
   <xacro:if value="$(arg hand_only)">
     <xacro:include filename="$(find moveit_resources_franka_panda_description)/urdf/hand.xacro"/>
-    <xacro:hand ns="$(arg arm_id)" rpy="0 0 ${-pi/4}" connected_to="$(arg arm_id)_link8" safety_distance="0.03"/>
+    <xacro:hand ns="$(arg arm_id)" rpy="0 0 0" connected_to="$(arg arm_id)_link8" safety_distance="0.03"/>
   </xacro:if>
   <xacro:if value="$(arg hand_realsense)">
@@ -18,10 +18,10 @@
     <xacro:include filename="$(find moveit_resources_franka_panda_description)/urdf/hand.xacro"/>
     <xacro:realsense_mount parent="$(arg arm_id)_link8">
-      <origin xyz="0 0 -0.0025" rpy="${radians(180)} 0 ${radians(180)}"/>
+      <origin xyz="0 0 0" rpy="${radians(180)} 0 ${radians(180)}"/>
     </xacro:realsense_mount>
     <xacro:sensor_d435 parent="camera_link" name="realsense">
-      <origin xyz="0 0 0" rpy="0 ${radians(-90)} ${radians(180)}"/>
+      <origin xyz="-0.015 0 0.005" rpy="0 ${radians(-90)} ${radians(180)}"/>
     </xacro:sensor_d435>
-    <xacro:hand ns="$(arg arm_id)" rpy="0 0 ${-pi/4}" connected_to="gripper_link" safety_distance="0.03"/>
+    <xacro:hand ns="$(arg arm_id)" rpy="0 0 0" connected_to="gripper_link" safety_distance="0.03"/>
   </xacro:if>
   <xacro:include filename="$(find moveit_resources_franka_panda_description)/urdf/panda_arm.ros2_control.xacro"/>
