Commit message: fix bug

File: franka_panda_description/urdf/panda_arm.urdf.xacro (robot description, xacro)
@@ -17,6 +17,10 @@
     <xacro:include filename="$(find realsense2_description)/urdf/_d435.urdf.xacro"/>
     <xacro:include filename="$(find moveit_resources_franka_panda_description)/urdf/hand.xacro"/>
-    <xacro:realsense_mount parent="panda_link8" xyz="0 0 -0.0025" rpy="${radians(180)} 0 ${radians(180)}"/>
-    <xacro:sensor_d435 parent="camera_link" xyz="0 0 0" rpy="0 ${radians(-90)} ${radians(180)}"/>
+    <xacro:realsense_mount parent="panda_link8">
+      <origin xyz="0 0 -0.0025" rpy="${radians(180)} 0 ${radians(180)}"/>
+    </xacro:realsense_mount>
+    <xacro:sensor_d435 parent="camera_link">
+      <origin xyz="0 0 0" rpy="0 ${radians(-90)} ${radians(180)}"/>
+    </xacro:sensor_d435>
     <xacro:hand ns="$(arg arm_id)" rpy="0 0 ${-pi/4}" connected_to="gripper_link" safety_distance="0.03"/>
   </xacro:if>

File: franka_panda_description/urdf/realsense_mount.xacro (robot description, xacro)
@@ -1,10 +1,9 @@
 <?xml version='1.0' encoding='utf-8'?>
 <robot name="realsense_mount" xmlns:xacro="http://ros.org/wiki/xacro">
-	<xacro:macro name="realsense_mount" params="parent">
+	<xacro:macro name="realsense_mount" params="parent *origin">
 		<joint name="arm_joint" type="fixed">
 			<parent link="${parent}"/>
 			<child link="arm_link"/>
 			<origin xyz="0 0 0.0025" rpy="0 0 0"/>
-			<axis xyz="0.0 0.0 1.0"/>
 		</joint>
 		<link name="mount_link">
@@ -26,5 +25,4 @@
 			<child link="gripper_link"/>
 			<origin xyz="0 0 -0.0025" rpy="0 0 0"/>
-			<axis xyz="0.0 0.0 1.0"/>
 		</joint>
 		<link name="gripper_link">
@@ -35,5 +33,4 @@
 			<child link="camera_link"/>
 			<origin xyz="0.06 0 0" rpy="0 0 0"/>
-			<axis xyz="0.0 0.0 1.0"/>
 		</joint>
 		<link name="camera_link">

Commit message: update realsense mount

File: franka_panda_description/urdf/panda_arm.urdf.xacro (robot description, xacro)
@@ -21,5 +21,5 @@
     </xacro:realsense_mount>
     <xacro:sensor_d435 parent="camera_link" name="realsense">
-      <origin xyz="-0.015 0 0.005" rpy="0 ${radians(-90)} ${radians(180)}"/>
+      <origin xyz="-0.0125 0 0.01" rpy="0 ${radians(-90)} ${radians(180)}"/>
     </xacro:sensor_d435>
     <xacro:hand ns="$(arg arm_id)" rpy="0 0 0" connected_to="gripper_link" safety_distance="0.03"/>

Commit message: add robotiq gripper

File: franka_panda_description/urdf/panda_arm.urdf.xacro (robot description, xacro)
@@ -2,6 +2,7 @@
 <robot xmlns:xacro="http://www.ros.org/wiki/xacro" name="panda">
   <xacro:arg name="arm_id" default="panda"/> <!-- Name of this panda -->
-  <xacro:arg name="hand_only" default="false"/> <!-- Should a franka_gripper be mounted at the flange?" -->
-  <xacro:arg name="hand_realsense" default="false"/> <!-- Should a franka_gripper and realsense be mounted at the flange?" -->
+  <xacro:arg name="panda_gripper" default="false"/> <!-- Should a franka_gripper be mounted at the flange?" -->
+  <xacro:arg name="panda_gripper_realsense" default="false"/> <!-- Should a franka_gripper and realsense be mounted at the flange?" -->
+  <xacro:arg name="robotiq_gripper" default="false"/> <!-- Should a robotiq gripper be mounted at the flange?" -->
   <xacro:arg name="robot_ip" default=""/> <!-- IP address or hostname of the robot" -->
   <xacro:arg name="use_fake_hardware" default="false"/>
@@ -9,9 +10,9 @@
   <xacro:include filename="$(find moveit_resources_franka_panda_description)/urdf/panda_arm.xacro"/>
   <xacro:panda_arm arm_id="$(arg arm_id)" safety_distance="0.03"/>
-  <xacro:if value="$(arg hand_only)">
+  <xacro:if value="$(arg panda_gripper)">
     <xacro:include filename="$(find moveit_resources_franka_panda_description)/urdf/hand.xacro"/>
     <xacro:hand ns="$(arg arm_id)" rpy="0 0 0" connected_to="$(arg arm_id)_link8" safety_distance="0.03"/>
   </xacro:if>
-  <xacro:if value="$(arg hand_realsense)">
+  <xacro:if value="$(arg panda_gripper_realsense)">
     <xacro:include filename="$(find moveit_resources_franka_panda_description)/urdf/realsense_mount.xacro"/>
     <xacro:include filename="$(find moveit_resources_franka_panda_description)/urdf/_d435.urdf.xacro"/>
@@ -23,5 +24,10 @@
       <origin xyz="-0.0125 0 0.01" rpy="0 ${radians(-90)} ${radians(180)}"/>
     </xacro:sensor_d435>
-    <xacro:hand ns="$(arg arm_id)" rpy="0 0 0" connected_to="gripper_link" safety_distance="0.03"/>
+  </xacro:if>
+  <xacro:if value="$(arg robotiq_gripper)">
+    <xacro:include filename="$(find robotiq_description)/urdf/robotiq_gripper_macro.urdf.xacro" />
+    <xacro:robotiq_gripper name="RobotiqGripperHardwareInterface" prefix="" parent="$(arg arm_id)_link8" use_fake_hardware="$(arg use_fake_hardware)">
+	<origin xyz="0 0 0" rpy="0 0 ${radians(-45)}" />
+    </xacro:robotiq_gripper>
   </xacro:if>
   <xacro:include filename="$(find moveit_resources_franka_panda_description)/urdf/panda_arm.ros2_control.xacro"/>

Commit message: clean description

File: franka_panda_description/urdf/panda_arm.urdf.xacro (robot description, xacro)
@@ -2,6 +2,4 @@
 <robot xmlns:xacro="http://www.ros.org/wiki/xacro" name="panda">
   <xacro:arg name="arm_id" default="panda"/> <!-- Name of this panda -->
-  <xacro:arg name="hand_only" default="false"/> <!-- Should a franka_gripper be mounted at the flange?" -->
-  <xacro:arg name="hand_realsense" default="false"/> <!-- Should a franka_gripper and realsense be mounted at the flange?" -->
   <xacro:arg name="robot_ip" default=""/> <!-- IP address or hostname of the robot" -->
   <xacro:arg name="use_fake_hardware" default="false"/>
@@ -9,20 +7,15 @@
   <xacro:include filename="$(find moveit_resources_franka_panda_description)/urdf/panda_arm.xacro"/>
   <xacro:panda_arm arm_id="$(arg arm_id)" safety_distance="0.03"/>
-  <xacro:if value="$(arg hand_only)">
-    <xacro:include filename="$(find moveit_resources_franka_panda_description)/urdf/hand.xacro"/>
-    <xacro:hand ns="$(arg arm_id)" rpy="0 0 0" connected_to="$(arg arm_id)_link8" safety_distance="0.03"/>
-  </xacro:if>
-  <xacro:if value="$(arg hand_realsense)">
-    <xacro:include filename="$(find moveit_resources_franka_panda_description)/urdf/realsense_mount.xacro"/>
-    <xacro:include filename="$(find realsense2_description)/urdf/_d435.urdf.xacro"/>
-    <xacro:include filename="$(find moveit_resources_franka_panda_description)/urdf/hand.xacro"/>
-    <xacro:realsense_mount parent="$(arg arm_id)_link8">
-      <origin xyz="0 0 0" rpy="${radians(180)} 0 ${radians(180)}"/>
-    </xacro:realsense_mount>
-    <xacro:sensor_d435 parent="camera_link" name="realsense">
-      <origin xyz="-0.015 0 0.005" rpy="0 ${radians(-90)} ${radians(180)}"/>
-    </xacro:sensor_d435>
-    <xacro:hand ns="$(arg arm_id)" rpy="0 0 0" connected_to="gripper_link" safety_distance="0.03"/>
-  </xacro:if>
+  <xacro:include filename="$(find robotiq_description)/urdf/robotiq_gripper_macro.urdf.xacro" />
+  <xacro:robotiq_gripper name="RobotiqGripperHardwareInterface" prefix="" parent="$(arg arm_id)_link8" use_fake_hardware="$(arg use_fake_hardware)">
+	<origin xyz="0 0 0" rpy="0 0 ${radians(-45)}" />
+  </xacro:robotiq_gripper>
+  <!-- Add an additional link to plan with. Oriented like the Panda ee_link frame. -->
+  <joint name="robotiq_gripper_tip_link_joint" type="fixed">
+    <parent link="robotiq_85_base_link"/>
+    <child link="robotiq_gripper_tip_link"/>
+    <origin rpy="0.0 0.0 0.0" xyz="0.246 0.0 0.0"/>
+  </joint>
+  <link name="robotiq_gripper_tip_link"/>
   <xacro:include filename="$(find moveit_resources_franka_panda_description)/urdf/panda_arm.ros2_control.xacro"/>
   <xacro:panda_arm_ros2_control ns="$(arg arm_id)" robot_ip="$(arg robot_ip)" use_fake_hardware="$(arg use_fake_hardware)" fake_sensor_commands="$(arg fake_sensor_commands)"/>

Commit message: fix tip link

File: franka_panda_description/urdf/panda_arm.urdf.xacro (robot description, xacro)
@@ -15,5 +15,5 @@
     <parent link="robotiq_85_base_link"/>
     <child link="robotiq_gripper_tip_link"/>
-    <origin rpy="0.0 0.0 0.0" xyz="0.246 0.0 0.0"/>
+    <origin rpy="0.0 0.0 0.0" xyz="0.0 0.0 0.16"/>
   </joint>
   <link name="robotiq_gripper_tip_link"/>
